File: BCPEHUB1/BCPEHUB1.sch (KiCad schematic (older format))
At the start: 32 parts, among them J1 Conn_01x02_Female, J10 Conn_01x05_Female, J4 Conn_01x02_Female, U1 TP4056, U2 DW01, U3 FS8205A, U4 ESP32-WROOM-32D, U5 BMP180, U6 HTU21DSMD

Commit message: Add files via upload
Parts:
- removed C5: 100n, Capacitor_SMD:C_1210_3225Metric_Pad1.33x2.70mm_HandSolder, symbol Device:C
- removed QA1, QB1: NTJD4401NT1, eec:On_Semiconductor-NTJD4401NT1-Manufacturer_Recommended, symbol eec:NTJD4401NT1
- removed R10, R11, R12, R13: 10k, Resistor_SMD:R_1210_3225Metric_Pad1.30x2.65mm_HandSolder, symbol Device:R
- removed U5: BMP180, SparkFun-Sensors:BMP180, symbol SparkFun-Sensors:BMP180
- removed U6: HTU21DSMD, SparkFun-Sensors:HTU21D, symbol SparkFun-Sensors:HTU21DSMD
- added J11, J13: Conn_01x04_Female, Connector_JST:JST_XH_B4B-XH-A_1x04_P2.50mm_Vertical, symbol Connector:Conn_01x04_Female
- added J20: Conn_01x03_Female, Connector_JST:JST_XH_B4B-XH-A_1x04_P2.50mm_Vertical, symbol Connector:Conn_01x03_Female
- C1: footprint Capacitor_THT:CP_Radial_D10.0mm_P2.50mm -> Capacitor_THT:CP_Radial_D4.0mm_P2.00mm
- C2: footprint Capacitor_SMD:C_0603_1608Metric_Pad1.08x0.95mm_HandSolder -> Capacitor_THT:C_Disc_D3.8mm_W2.6mm_P2.50mm
- C3, C4: footprint Capacitor_SMD:CP_Elec_8x6.5 -> Capacitor_THT:C_Radial_D10.0mm_H12.5mm_P5.00mm
- D1, D2: footprint LED_SMD:LED_0603_1608Metric_Pad1.05x0.95mm_HandSolder -> LED_THT:LED_D1.8mm_W3.3mm_H2.4mm
- J1, J4: footprint Connector_JST:JST_EH_B2B-EH-A_1x02_P2.50mm_Vertical -> Connector_JST:JST_XH_B2B-XH-A_1x02_P2.50mm_Vertical
- R1, R2, R3, R4, R5, R6, R7, R8, R9: footprint Resistor_SMD:R_1210_3225Metric_Pad1.30x2.65mm_HandSolder -> Resistor_THT:R_Axial_DIN0204_L3.6mm_D1.6mm_P7.62mm_Horizontal
- R15: footprint (none) -> Resistor_THT:R_Axial_DIN0204_L3.6mm_D1.6mm_P7.62mm_Horizontal
Connections:
- net OUT- is gone; now on net GND: C1.2
- net 3,3V+: now also J11.4 (Pin_4), J13.4 (Pin_4)
- net GND: now also J11.3 (Pin_3), J13.3 (Pin_3), J20.3 (Pin_3)
- net at U4.21 (SDO/SD0): now also J11.1 (Pin_1), J13.1 (Pin_1)
- net at U4.22 (SDI/SD1): now also J11.2 (Pin_2), J13.2 (Pin_2)
- net at U4.34 (RXD0/IO3): now also J20.2 (Pin_2)
- net at U4.35 (TXD0/IO1): now also J20.1 (Pin_1)
- no-connect marks 33 -> 31
Other:
- note added: "Programovací konektor"
