File: BCPEHUB1/BCPEHUB2.sch (KiCad schematic (older format))
At the start: 36 parts, among them J1 Conn_01x02_Female, J10 Conn_01x05_Female, J11 Conn_01x04_Female, J12 Conn_01x04_Male, J13 Conn_01x04_Female, J14 Conn_01x04_Male, J4 Conn_01x02_Female, U1 TP4056, U2 DW01, U3 FS8205A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

Commit message: Add files via upload
Other:
- note added: "Nastavení odporu R3\npro nabíjení proudem\n130mA až 1A"
- note added: "\n"
- note removed: "+5"
- note removed: "Set Charging\n Current to 130ma\n"
Changed lines of the file:
@@
 encoding utf-8
 Sheet 1 1
-Title ""
-Date ""
-Rev ""
+Title "Enviromental sensor measuring with ESP32"
+Date "2021-07-17"
+Rev "B"
 Comp ""
 Comment1 ""
@@
 Text GLabel 9400 1500 2    39   Input ~ 0
 BAT+
-Text Notes 2300 1800 0    60   ~ 0
-+5
 $Comp
 L Device:R R8
@@
 Text GLabel 9400 2600 2    39   Input ~ 0
 GND
-Text Notes 5050 2100 0    39   ~ 0
-Set Charging\n Current to 130ma\n
+Text Notes 4750 2100 0    39   ~ 0
+Nastavení odporu R3\npro nabíjení proudem\n130mA až 1A
 Wire Wire Line
 	3200 1500 3500 1500
@@
 Wire Wire Line
 	5950 2400 5950 2100
-Text Notes 6000 1700 0    60   ~ 0
-ceramic cap\n
 $Comp
 L fs8205a:FS8205A U3
@@
 Connection ~ 3900 1450
 Text Notes 1950 2100 0    60   ~ 0
-ceramic cap\n
+\n
 Text Notes 8550 1800 0    60   ~ 0
 ceramic cap\n
