File: BCPEHUB1/BCPEHUB3.sch (KiCad schematic (older format))
At the start: 25 parts, among them J1 Conn_01x02_Female, J10 Conn_01x05_Female, J11 Conn_01x04_Female, J13 Conn_01x04_Female, J4 Conn_01x02_Female, U1 TP4056, U2 DW01, U3 FS8205A, U4 ESP32-WROOM-32D

Commit message: Add files via upload
Parts:
- C1: footprint Capacitor_THT:CP_Radial_D10.0mm_P2.50mm -> Capacitor_THT:CP_Radial_D4.0mm_P2.00mm
- C2: footprint Capacitor_SMD:C_0603_1608Metric_Pad1.08x0.95mm_HandSolder -> Capacitor_THT:C_Disc_D3.8mm_W2.6mm_P2.50mm
- C3, C4: footprint Capacitor_SMD:CP_Elec_8x6.5 -> Capacitor_THT:C_Radial_D10.0mm_H12.5mm_P5.00mm
- D1, D2: footprint LED_SMD:LED_0603_1608Metric_Pad1.05x0.95mm_HandSolder -> LED_THT:LED_D1.8mm_W3.3mm_H2.4mm
- J1, J4: footprint Connector_JST:JST_EH_B2B-EH-A_1x02_P2.50mm_Vertical -> Connector_JST:JST_XH_B2B-XH-A_1x02_P2.50mm_Vertical
- J11, J13: footprint (none) -> Connector_JST:JST_XH_B4B-XH-AM_1x04_P2.50mm_Vertical
- R1, R2, R3, R4, R5, R6, R7, R8, R9: footprint Resistor_SMD:R_1210_3225Metric_Pad1.30x2.65mm_HandSolder -> Resistor_THT:R_Axial_DIN0204_L3.6mm_D1.6mm_P7.62mm_Horizontal
- R15: footprint (none) -> Resistor_THT:R_Axial_DIN0204_L3.6mm_D1.6mm_P7.62mm_Horizontal
Changed lines of the file:
@@
 encoding utf-8
 Sheet 1 1
-Title ""
-Date ""
-Rev ""
+Title "Enviromental sensor measurement with ESP32"
+Date "2021-07-17"
+Rev "C"
 Comp ""
 Comment1 ""
@@
 F 0 "R5" V 3730 1500 50  0000 C CNN
 F 1 "1k" V 3650 1500 50  0000 C CNN
-F 2 "Resistor_SMD:R_1210_3225Metric_Pad1.30x2.65mm_HandSolder" V 3580 1500 50  0001 C CNN
+F 2 "Resistor_THT:R_Axial_DIN0204_L3.6mm_D1.6mm_P7.62mm_Horizontal" V 3580 1500 50  0001 C CNN
 F 3 "" H 3650 1500 50  0001 C CNN
 	1    3650 1500
@@
 F 0 "C2" H 2675 2150 50  0000 L CNN
 F 1 "0.1uF" H 2675 1950 50  0000 L CNN
-F 2 "Capacitor_SMD:C_0603_1608Metric_Pad1.08x0.95mm_HandSolder" H 2688 1900 50  0001 C CNN
+F 2 "Capacitor_THT:C_Disc_D3.8mm_W2.6mm_P2.50mm" H 2688 1900 50  0001 C CNN
 F 3 "" H 2650 2050 50  0001 C CNN
 	1    2650 2050
@@
 F 0 "D2" H 3050 1900 50  0000 C CNN
 F 1 "LED" H 3050 1700 50  0000 C CNN
-F 2 "LED_SMD:LED_0603_1608Metric_Pad1.05x0.95mm_HandSolder" H 3050 1800 50  0001 C CNN
+F 2 "LED_THT:LED_D1.8mm_W3.3mm_H2.4mm" H 3050 1800 50  0001 C CNN
 F 3 "" H 3050 1800 50  0001 C CNN
 	1    3050 1800
@@
 F 0 "R6" V 3680 1800 50  0000 C CNN
 F 1 "1k" V 3600 1800 50  0000 C CNN
-F 2 "Resistor_SMD:R_1210_3225Metric_Pad1.30x2.65mm_HandSolder" V 3530 1800 50  0001 C CNN
+F 2 "Resistor_THT:R_Axial_DIN0204_L3.6mm_D1.6mm_P7.62mm_Horizontal" V 3530 1800 50  0001 C CNN
 F 3 "" H 3600 1800 50  0001 C CNN
 	1    3600 1800
@@
 F 0 "D1" H 3050 1600 50  0000 C CNN
 F 1 "LED" H 3050 1400 50  0000 C CNN
-F 2 "LED_SMD:LED_0603_1608Metric_Pad1.05x0.95mm_HandSolder" H 3050 1500 50  0001 C CNN
+F 2 "LED_THT:LED_D1.8mm_W3.3mm_H2.4mm" H 3050 1500 50  0001 C CNN
 F 3 "" H 3050 1500 50  0001 C CNN
 	1    3050 1500
@@
 F 0 "R7" V 5480 1750 50  0000 C CNN
 F 1 "10k" V 5400 1750 50  0000 C CNN
-F 2 "Resistor_SMD:R_1210_3225Metric_Pad1.30x2.65mm_HandSolder" V 5330 1750 50  0001 C CNN
+F 2 "Resistor_THT:R_Axial_DIN0204_L3.6mm_D1.6mm_P7.62mm_Horizontal" V 5330 1750 50  0001 C CNN
 F 3 "" H 5400 1750 50  0001 C CNN
 	1    5400 1750
@@
 F 0 "R8" V 6830 1950 50  0000 C CNN
 F 1 "1k" V 6750 1950 50  0000 C CNN
-F 2 "Resistor_SMD:R_1210_3225Metric_Pad1.30x2.65mm_HandSolder" V 6680 1950 50  0001 C CNN
+F 2 "Resistor_THT:R_Axial_DIN0204_L3.6mm_D1.6mm_P7.62mm_Horizontal" V 6680 1950 50  0001 C CNN
 F 3 "" H 6750 1950 50  0001 C CNN
 	1    6750 1950
@@
 F 0 "C4" H 8325 1900 50  0000 L CNN
 F 1 "0.1uF" H 8325 1700 50  0000 L CNN
-F 2 "Capacitor_SMD:CP_Elec_8x6.5" H 8338 1650 50  0001 C CNN
+F 2 "Capacitor_THT:C_Radial_D10.0mm_H12.5mm_P5.00mm" H 8338 1650 50  0001 C CNN
 F 3 "" H 8300 1800 50  0001 C CNN
 	1    8300 1800
@@
 F 0 "R9" V 8880 1500 50  0000 C CNN
 F 1 "100" V 8800 1500 50  0000 C CNN
-F 2 "Resistor_SMD:R_1210_3225Metric_Pad1.30x2.65mm_HandSolder" V 8730 1500 50  0001 C CNN
+F 2 "Resistor_THT:R_Axial_DIN0204_L3.6mm_D1.6mm_P7.62mm_Horizontal" V 8730 1500 50  0001 C CNN
 F 3 "" H 8800 1500 50  0001 C CNN
 	1    8800 1500
@@
 F 0 "C3" H 5975 2050 50  0000 L CNN
 F 1 "10uF" H 5975 1850 50  0000 L CNN
-F 2 "Capacitor_SMD:CP_Elec_8x6.5" H 5988 1800 50  0001 C CNN
+F 2 "Capacitor_THT:C_Radial_D10.0mm_H12.5mm_P5.00mm" H 5988 1800 50  0001 C CNN
 F 3 "" H 5950 1950 50  0001 C CNN
 	1    5950 1950
@@
 F 0 "R3" H 5470 6946 50  0000 L CNN
 F 1 "10k" H 5470 6855 50  0000 L CNN
-F 2 "Resistor_SMD:R_1210_3225Metric_Pad1.30x2.65mm_HandSolder" V 5330 6900 50  0001 C CNN
+F 2 "Resistor_THT:R_Axial_DIN0204_L3.6mm_D1.6mm_P7.62mm_Horizontal" V 5330 6900 50  0001 C CNN
 F 3 "~" H 5400 6900 50  0001 C CNN
 	1    5400 6900
@@
 F 0 "R4" H 5470 7246 50  0000 L CNN
 F 1 "10k" H 5470 7155 50  0000 L CNN
-F 2 "Resistor_SMD:R_1210_3225Metric_Pad1.30x2.65mm_HandSolder" V 5330 7200 50  0001 C CNN
+F 2 "Resistor_THT:R_Axial_DIN0204_L3.6mm_D1.6mm_P7.62mm_Horizontal" V 5330 7200 50  0001 C CNN
 F 3 "~" H 5400 7200 50  0001 C CNN
 	1    5400 7200
@@
 F 0 "R1" H 5470 6096 50  0000 L CNN
 F 1 "10k" H 5470 6005 50  0000 L CNN
-F 2 "Resistor_SMD:R_1210_3225Metric_Pad1.30x2.65mm_HandSolder" V 5330 6050 50  0001 C CNN
+F 2 "Resistor_THT:R_Axial_DIN0204_L3.6mm_D1.6mm_P7.62mm_Horizontal" V 5330 6050 50  0001 C CNN
 F 3 "~" H 5400 6050 50  0001 C CNN
 	1    5400 6050
@@
 F 0 "R2" H 5470 6396 50  0000 L CNN
 F 1 "10k" H 5470 6305 50  0000 L CNN
-F 2 "Resistor_SMD:R_1210_3225Metric_Pad1.30x2.65mm_HandSolder" V 5330 6350 50  0001 C CNN
+F 2 "Resistor_THT:R_Axial_DIN0204_L3.6mm_D1.6mm_P7.62mm_Horizontal" V 5330 6350 50  0001 C CNN
 F 3 "~" H 5400 6350 50  0001 C CNN
 	1    5400 6350
@@
 F 0 "J1" H 1778 1876 50  0000 L CNN
 F 1 "Conn_01x02_Female" H 1778 1785 50  0001 R BNN
-F 2 "Connector_JST:JST_EH_B2B-EH-A_1x02_P2.50mm_Vertical" H 1750 1900 50  0001 C CNN
+F 2 "Connector_JST:JST_XH_B2B-XH-A_1x02_P2.50mm_Vertical" H 1750 1900 50  0001 C CNN
 F 3 "~" H 1750 1900 50  0001 C CNN
 	1    1750 1900
@@
 F 0 "C1" V 3368 4046 50  0000 L CNN
 F 1 "10uF" V 3368 3955 50  0000 R CNN
-F 2 "Capacitor_THT:CP_Radial_D10.0mm_P2.50mm" H 3288 3850 50  0001 C CNN
+F 2 "Capacitor_THT:CP_Radial_D4.0mm_P2.00mm" H 3288 3850 50  0001 C CNN
 F 3 "~" H 3250 4000 50  0001 C CNN
 	1    3250 4000
@@
 F 0 "J4" H 9578 1726 50  0000 L TNN
 F 1 "Conn_01x02_Female" H 9578 1635 50  0001 R BNN
-F 2 "Connector_JST:JST_EH_B2B-EH-A_1x02_P2.50mm_Vertical" H 9550 1750 50  0001 C CNN
+F 2 "Connector_JST:JST_XH_B2B-XH-A_1x02_P2.50mm_Vertical" H 9550 1750 50  0001 C CNN
 F 3 "~" H 9550 1750 50  0001 C CNN
 	1    9550 1750
@@
 F 0 "R15" H 3470 3746 50  0000 L CNN
 F 1 "10k" H 3470 3655 50  0000 L CNN
-F 2 "" V 3330 3700 50  0001 C CNN
+F 2 "Resistor_THT:R_Axial_DIN0204_L3.6mm_D1.6mm_P7.62mm_Horizontal" V 3330 3700 50  0001 C CNN
 F 3 "~" H 3400 3700 50  0001 C CNN
 	1    3400 3700
@@
 F 0 "J11" H 2442 4367 50  0000 C CNN
 F 1 "Conn_01x04_Female" H 2442 4366 50  0001 C CNN
-F 2 "" H 2550 4700 50  0001 C CNN
+F 2 "Connector_JST:JST_XH_B4B-XH-AM_1x04_P2.50mm_Vertical" H 2550 4700 50  0001 C CNN
 F 3 "~" H 2550 4700 50  0001 C CNN
 	1    2550 4700
@@
 F 0 "J13" H 2492 5667 50  0000 C CNN
 F 1 "Conn_01x04_Female" H 2492 5666 50  0001 C CNN
-F 2 "" H 2600 6000 50  0001 C CNN
+F 2 "Connector_JST:JST_XH_B4B-XH-AM_1x04_P2.50mm_Vertical" H 2600 6000 50  0001 C CNN
 F 3 "~" H 2600 6000 50  0001 C CNN
 	1    2600 6000
