File: BCPEHUB1/_autosave-BCPEHUB1.kicad_pcb (KiCad board)
At the start: 2 copper layers, 100.3 x 48.3 mm, 30 parts, among them J1 Conn_01x02_Female, J10 Conn_01x05_Female, J11 Conn_01x04_Female, J13 Conn_01x04_Female, J20 Conn_01x03_Female, J4 Conn_01x02_Female, U1 TP4056, U2 DW01, U3 FS8205A, U4 ESP32-WROOM-32D

Commit message: Add files via upload
Parts:
- J11, J13: footprint Connector_JST:JST_XH_B4B-XH-AM_1x04_P2.50mm_Vertical -> Connector_JST:JST_XH_B4B-XH-A_1x04_P2.50mm_Vertical
- J20: footprint Connector_JST:JST_XH_B3B-XH-AM_1x03_P2.50mm_Vertical -> Connector_JST:JST_XH_B4B-XH-A_1x04_P2.50mm_Vertical
